File: ieee_pcb_workshop.kicad_sch (KiCad schematic)
At the start: 48 parts, among them J1 Conn_01x10, J2 Conn_01x10, J3 ICSP, J4 USB_B_Micro, U1 ATmega32U4-A, Y1 16MHz

Commit message: add 01 lecture
Other:
- note removed: "PERIPHERAL"
- note removed: "TODO"
Changed lines of the file:
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@@
-    (fill (type none))
-  )
-  (rectangle (start 17.78 29.845) (end 113.03 74.295)
-    (stroke (width 0) (type default))
     (fill (type none))
   )
@@
     (effects (font (size 1.27 1.27)) (justify left bottom))
   )
-  (text "TODO" (at 60.96 53.34 0)
-    (effects (font (size 1.27 1.27)) (justify left bottom))
-  )
   (text "D5" (at 93.98 125.73 0)
     (effects (font (size 1.27 1.27)) (justify left bottom))
@@
     (effects (font (size 1.27 1.27)) (justify left bottom))
   )
-  (text "PERIPHERAL" (at 59.055 28.575 0)
-    (effects (font (size 1.27 1.27)) (justify left bottom))
-  )
