File: ieee_pcb_workshop.kicad_pcb (KiCad board)
At the start: 2 copper layers, 105 x 40 mm, 50 parts, among them J1 Conn_01x10, J2 Conn_01x10, J3 ICSP, J4 USB_B_Micro, U1 ATmega32U4-A, Y1 16MHz

Commit message: add 01 lecture
Parts:
- removed the G*** at (132.0, 161.5)
- added G***: LOGO, LOGO, F.Cu at (126.0, 162.0)
- added G***: LOGO, LOGO, F.Cu at (147.9, 175.5)
- moved G*** 2.66 mm to (142.2, 161.8)
Routing:
- net +5V: track 142.4 -> 143.9 mm, vias 31 -> 30
- net GND: vias 8 -> 9
Other:
- board size 105 x 40 mm -> 102 x 40 mm

Commit message: day 1 slides
Routing:
- net +5V: track 143.9 -> 142.6 mm
- net GND: vias 9 -> 11
Changed lines of the file:
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@@
     (grid_origin 82 135)
     (pcbplotparams
-      (layerselection 0x00010f0_ffffffff)
+      (layerselection 0x00010fc_ffffffff)
       (plot_on_all_layers_selection 0x0000000_00000000)
       (disableapertmacros false)
@@
       (psa4output false)
       (plotreference true)
-      (plotvalue true)
+      (plotvalue false)
       (plotinvisibletext false)
       (sketchpadsonfab false)
-      (subtractmaskfromsilk false)
+      (subtractmaskfromsilk true)
       (outputformat 1)
       (mirror false)
@@
   (segment (start 84.125 145) (end 85 145) (width 0.25) (layer "F.Cu") (net 1))
   (segment (start 54.2 132.5) (end 50.13 128.43) (width 0.4) (layer "F.Cu") (net 1))
-  (segment (start 62.26 139.04) (end 63.285 139.04) (width 0.4) (layer "F.Cu") (net 1))
   (segment (start 120.875 155.875) (end 121 156) (width 0.25) (layer "F.Cu") (net 1))
   (segment (start 81.125 135) (end 80.25 135.875) (width 0.25) (layer "F.Cu") (net 1))
@@
   (segment (start 60.2 143) (end 60.2 143) (width 0.4) (layer "F.Cu") (net 1))
   (segment (start 126.25 147) (end 127.25 147) (width 0.25) (layer "F.Cu") (net 1))
-  (segment (start 63.285 139.04) (end 63.41 139.165) (width 0.4) (layer "F.Cu") (net 1))
   (segment (start 108.75 137) (end 108.5 137.25) (width 0.25) (layer "F.Cu") (net 1))
   (segment (start 61.15 150.75) (end 61.15 155.131) (width 0.4) (layer "F.Cu") (net 1))
@@
   (segment (start 81.9 134.9) (end 82 135) (width 0.4) (layer "B.Cu") (net 1))
   (via (at 58.6 133.2) (size 0.8) (drill 0.4) (layers "F.Cu" "B.Cu") (free) (net 2))
+  (via (at 60.8 148.85) (size 0.8) (drill 0.4) (layers "F.Cu" "B.Cu") (free) (net 2))
   (via (at 67.4 156.4) (size 0.8) (drill 0.4) (layers "F.Cu" "B.Cu") (free) (net 2))
+  (via (at 59 145.7) (size 0.8) (drill 0.4) (layers "F.Cu" "B.Cu") (free) (net 2))
   (via (at 54 142) (size 0.8) (drill 0.4) (layers "F.Cu" "B.Cu") (free) (net 2))
   (via (at 67.8 142.2) (size 0.8) (drill 0.4) (layers "F.Cu" "B.Cu") (free) (net 2))
