File: kicad/ieee_pcb_workshop.kicad_pcb (KiCad board)
At the start: 2 copper layers, 102 x 40 mm, 51 parts, among them J1 Conn_01x10, J2 Conn_01x10, J3 ICSP, J4 USB_B_Micro, U1 ATmega32U4-A, Y1 16MHz

Commit message: add starter code
Parts:
- removed the G*** at (147.9, 175.5)
Other:
- board text added: "JLCJLCJLCJLC"
- board text added: "rev1 | 04.10.24"
- board text removed: "rev1 | 03.20.24"
